Commit message: update my urdf

File: description_urdf/robot_2/single_joint.urdf (robot description, URDF)
Before this commit: robot Single_Joint, 2 links, 1 joints
Links:
- link Link_2: geometry collision box size=1 5 0.5; visual box size=0.5 5 0.5

File: ros_control_ur5/urdf/ur5_ros_control.urdf (robot description, URDF)
Before this commit: robot ur5, 9 links, 8 joints
Links:
- link base_link: geometry collision mesh filename=package://ros_control_ur5/meshes/ur5/collision/base.stl; visual mesh filename=package://ros_control_ur5/meshes/ur5/visual/base.dae
- link forearm_link: geometry collision mesh filename=package://ros_control_ur5/meshes/ur5/collision/forearm.stl; visual mesh filename=package://ros_control_ur5/meshes/ur5/visual/forearm.dae
- link shoulder_link: geometry collision mesh filename=package://ros_control_ur5/meshes/ur5/collision/shoulder.stl; visual mesh filename=package://ros_control_ur5/meshes/ur5/visual/shoulder.dae
- link upper_arm_link: geometry collision mesh filename=package://ros_control_ur5/meshes/ur5/collision/upperarm.stl; visual mesh filename=package://ros_control_ur5/meshes/ur5/visual/upperarm.dae
- link wrist_1_link: geometry collision mesh filename=package://ros_control_ur5/meshes/ur5/collision/wrist1.stl; visual mesh filename=package://ros_control_ur5/meshes/ur5/visual/wrist1.dae
- link wrist_2_link: geometry collision mesh filename=package://ros_control_ur5/meshes/ur5/collision/wrist2.stl; visual mesh filename=package://ros_control_ur5/meshes/ur5/visual/wrist2.dae
- link wrist_3_link: geometry collision mesh filename=package://ros_control_ur5/meshes/ur5/collision/wrist3.stl; visual mesh filename=package://ros_control_ur5/meshes/ur5/visual/wrist3.dae
